File: Hardware/ST-Link-V2.1.kicad_pcb (KiCad board)
At the start: 2 copper layers, 13.9 x 35.8 mm, 42 parts, among them IC1 LP2992AIM5X-3.3, J1 USB_C_Receptacle, J2 Conn_01x05_Pin, J3 Conn_01x05_Pin, J4 Conn_01x04_Pin, Q1 S8050, U1 STM32F103C8T6, Y1 CSTCE12M0G55-R0

Commit message: Update Hardware
Parts:
- U1: value STM32F103C8T6 -> STM32F103CBT6
- Y1: value CSTCE12M0G55-R0 -> CSTCE8M0G55-R0
Changed lines of the file:
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@@
 		(tags "resistor")
 		(property "Reference" "R1"
-			(at 0 -1.43 360)
+			(at 0 -1.43 0)
 			(layer "F.SilkS")
 			(hide yes)
@@
 		)
 		(property "Value" "10K"
-			(at 0 1.43 360)
+			(at 0 1.43 0)
 			(layer "F.Fab")
 			(hide yes)
@@
 		(tags "capacitor")
 		(property "Reference" "C6"
-			(at 0 -1.43 360)
+			(at 0 -1.43 0)
 			(layer "F.SilkS")
 			(hide yes)
@@
 		)
 		(property "Value" "0.1uF"
-			(at 0 1.43 360)
+			(at 0 1.43 0)
 			(layer "F.Fab")
 			(hide yes)
@@
 		(tags "LED")
 		(property "Reference" "D2"
-			(at 0 -1.43 270)
+			(at 0 -1.43 -90)
 			(layer "F.SilkS")
 			(hide yes)
@@
 		)
 		(property "Value" "POWER"
-			(at 0 1.43 270)
+			(at 0 1.43 -90)
 			(layer "F.Fab")
 			(hide yes)
@@
 			)
 		)
-		(property "Value" "CSTCE12M0G55-R0"
+		(property "Value" "CSTCE8M0G55-R0"
 			(at 0 0 0)
 			(layer "F.SilkS")
@@
 			(layer "F.Fab")
 		)
+		(fp_text user "${REFERENCE}"
+			(at 0 0 0)
+			(layer "F.Fab")
+			(effects
+				(font
+					(size 1.27 1.27)
+					(thickness 0.254)
+				)
+			)
+		)
 		(pad "1" smd rect
 			(at -1.2 0)
@@
 		(tags "resistor")
 		(property "Reference" "R7"
-			(at 0 -1.43 270)
+			(at 0 -1.43 -90)
 			(layer "F.SilkS")
 			(hide yes)
@@
 		)
 		(property "Value" "10K"
-			(at 0 1.43 270)
+			(at 0 1.43 -90)
 			(layer "F.Fab")
 			(hide yes)
@@
 		(tags "LED")
 		(property "Reference" "D3"
-			(at 0 -1.43 270)
+			(at 0 -1.43 -90)
 			(layer "F.SilkS")
 			(hide yes)
@@
 		)
 		(property "Value" "LOAD"
-			(at 0 1.43 270)
+			(at 0 1.43 -90)
 			(layer "F.Fab")
 			(hide yes)
@@
 		(tags "resistor")
 		(property "Reference" "R17"
-			(at 0 -1.43 270)
+			(at 0 -1.43 -90)
 			(layer "F.SilkS")
 			(hide yes)
@@
 		)
 		(property "Value" "100R"
-			(at 0 1.43 270)
+			(at 0 1.43 -90)
 			(layer "F.Fab")
 			(hide yes)
@@
 		(tags "LQFP QFP")
 		(property "Reference" "U1"
-			(at 0 -5.85 270)
+			(at 0 -5.85 -90)
 			(layer "F.SilkS")
 			(hide yes)
@@
 			)
 		)
-		(property "Value" "STM32F103C8T6"
-			(at 0 5.85 270)
+		(property "Value" "STM32F103CBT6"
+			(at 0 5.85 -90)
 			(layer "F.Fab")
 			(hide yes)
@@
 		(tags "solder jumper open")
 		(property "Reference" "JP1"
-			(at 0 1.8 270)
+			(at 0 1.8 -90)
 			(layer "B.SilkS")
 			(hide yes)
@@
 		)
 		(property "Value" "BOOT0"
-			(at 0 -1.9 270)
+			(at 0 -1.9 -90)
 			(layer "B.Fab")
 			(hide yes)
@@
 		(tags "capacitor")
 		(property "Reference" "C7"
-			(at 0 1.43 270)
+			(at 0 1.43 -90)
 			(layer "B.SilkS")
 			(hide yes)
@@
 		)
 		(property "Value" "1uF"
-			(at 0 -1.43 270)
+			(at 0 -1.43 -90)
 			(layer "B.Fab")
 			(hide yes)
@@
 		(tags "resistor")
 		(property "Reference" "R11"
-			(at 0 1.43 270)
+			(at 0 1.43 -90)
 			(layer "B.SilkS")
 			(hide yes)
@@
 		)
 		(property "Value" "10K"
-			(at 0 -1.43 270)
+			(at 0 -1.43 -90)
 			(layer "B.Fab")
 			(hide yes)
@@
 			(layer "B.Fab")
 		)
+		(fp_text user "${REFERENCE}"
+			(at 0 0 -90)
+			(layer "B.Fab")
+			(effects
+				(font
+					(size 1.27 1.27)
+					(thickness 0.254)
+				)
+				(justify mirror)
+			)
+		)
 		(pad "1" smd rect
 			(at -1.25 0.95 180)
@@
 		(tags "capacitor")
 		(property "Reference" "C8"
-			(at 0 1.43 270)
+			(at 0 1.43 -90)
 			(layer "B.SilkS")
 			(hide yes)
@@
 		)
 		(property "Value" "1uF"
-			(at 0 -1.43 270)
+			(at 0 -1.43 -90)
 			(layer "B.Fab")
 			(hide yes)
@@
 		(tags "resistor")
 		(property "Reference" "R12"
-			(at 0 1.43 270)
+			(at 0 1.43 -90)
 			(layer "B.SilkS")
 			(hide yes)
@@
 		)
 		(property "Value" "100R"
-			(at 0 -1.43 270)
+			(at 0 -1.43 -90)
 			(layer "B.Fab")
 			(hide yes)
@@
 		(tags "resistor")
 		(property "Reference" "R14"
-			(at 0 1.43 360)
+			(at 0 1.43 0)
 			(layer "B.SilkS")
 			(hide yes)
@@
 		)
 		(property "Value" "100R"
-			(at 0 -1.43 360)
+			(at 0 -1.43 0)
 			(layer "B.Fab")
 			(hide yes)
@@
 		(tags "capacitor")
 		(property "Reference" "C9"
-			(at 0 1.43 360)
+			(at 0 1.43 0)
 			(layer "B.SilkS")
 			(hide yes)
@@
 		)
 		(property "Value" "10nF"
-			(at 0 -1.43 360)
+			(at 0 -1.43 0)
 			(layer "B.Fab")
 			(hide yes)
