File: Hardware/ST-Link-V2.1.kicad_sch (KiCad schematic)
At the start: 40 parts, among them IC1 LP2992AIM5X-3.3, J1 USB_C_Receptacle, J2 Conn_01x05_Pin, J3 Conn_01x05_Pin, J4 Conn_01x04_Pin, Q1 S8050, U1 STM32F103C8T6, Y1 CSTCE12M0G55-R0

Commit message: Update Hardware
Parts:
- U1: value STM32F103C8T6 -> STM32F103CBT6
- Y1: value CSTCE12M0G55-R0 -> CSTCE8M0G55-R0
Changed lines of the file:
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@@
 			)
 		)
-		(property "Value" "CSTCE12M0G55-R0"
+		(property "Value" "CSTCE8M0G55-R0"
 			(at 115.57 87.63 0)
 			(effects
@@
 			)
 		)
-		(property "Value" "STM32F103C8T6"
+		(property "Value" "STM32F103CBT6"
 			(at 54.2641 105.41 0)
 			(effects
